Commit message: add blender render recorder

File: panda_gym/assets/cup.urdf (robot description, URDF)
Before this commit: robot your_robot_name, 1 links, 0 joints
Links:
- link base_link: mass 0.5 -> 0

File: panda_gym/assets/plate.urdf (robot description, URDF)
Before this commit: robot your_robot_name, 1 links, 0 joints
Links:
- link base_link: mass 0.5 -> 0
